File: spirometer_design/Spiro/spiroBoardV2/microcontroller.sch (KiCad schematic (older format))
At the start: 40 parts, among them J2 USB_B_Mini, J4 Conn_01x11_Female, J5 Conn_02x03_Odd_Even, J6 Conn_01x07_Female, SW2 SW_Push, U3 ZTX690B-ND, U4 RT9261A-50GB, U5 ATmega32U4-MU, Y1 16MHz

Commit message: germany
Parts:
- U5: symbol MCU_Microchip_ATmega:ATmega32U4-MU -> spiroBoardV2-rescue:ATmega32U4-MU-MCU_Microchip_ATmega
Changed lines of the file:
@@
 EESchema Schematic File Version 4
-LIBS:spiroBoardV2-cache
 EELAYER 30 0
 EELAYER END
@@
 pressureSensorHigh
 $Comp
-L MCU_Microchip_ATmega:ATmega32U4-MU U?
+L spiroBoardV2-rescue:ATmega32U4-MU-MCU_Microchip_ATmega U?
 U 1 1 5D70EC65
 P 7700 3350
