File: spirometer_design/Spiro/spiroBoardV2/spiroBoardV2.kicad_pcb (KiCad board)
At the start: 2 copper layers, 66.1 x 88.5 mm, 71 parts, among them J1 Barrel_Jack_Switch, J2 USB_B_Mini, J3 Screw_Terminal_01x02, J4 Conn_01x11_Female, J5 Conn_02x03_Odd_Even, J6 Conn_01x07_Female, SW2 SW_Push, U1 INA168, U2 OPA340NA, U3 ZTX690B-ND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

Commit message: germany
Parts:
- removed Sol Discharge Switch: SW_Push_Open, SpiroParts:Slide_Switch_SPST_Through_Hole
- added SW1: SW_Push_Open, SpiroParts:Slide_Switch_SPST_Through_Hole, F.Cu at (123.4, 92.3)
- moved R10 2.00 mm to (118.5, 140.7), turned to 180 degrees
- moved D4 0.79 mm to (118.6, 142.7)
- moved C9 0.20 mm to (113.6, 137.9)
- renumbered HWB to JP1, PSH to TP1, PSL to TP2, 5V to TP5, solTog to TP6, SolGND to TP9
Routing:
- net /5V: track 202.7 -> 205.8 mm
- net Net-(R3-Pad2): track 11.1 -> 9.08 mm
- net Net-(C6-Pad2): track 18.8 -> 19.9 mm
- net GND: vias 16 -> 18
